File: latbox_cycloneV.kicad_pcb (KiCad board)
At the start: 4 copper layers, 130 x 100 mm, 194 parts, among them J101 GPIO0, J201 Conn_Coaxial, J202 Conn_Coaxial, J203 Conn_Coaxial, J204 Conn_Coaxial, J301 Conn_Coaxial, J302 Conn_Coaxial, J303 Conn_Coaxial, J304 Conn_Coaxial, J401 OUT1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

Commit message: Add markings
Signed-off-by: Benedikt Spranger <b.spranger@linutronix.de>
Parts:
- added G1: LOGO, eurovibes:LOGO, F.Cu at (174.0, 64.0)
Other:
- board text added: "DE0-nano-SoC Latencybox v0.1"
