File: latbox_cycloneV.kicad_sch (KiCad schematic)
At the start: 7 parts, among them J101 GPIO0

Commit message: Add markings
Signed-off-by: Benedikt Spranger <b.spranger@linutronix.de>
Parts:
- added G1: LOGO, eurovibes:LOGO, symbol eurovibes:LOGO
Changed lines of the file:
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@@
     (effects (font (size 1.27 1.27)) (justify right bottom))
+  )
+  (symbol (lib_id "eurovibes:LOGO") (at 280.67 162.56 0) (unit 1)
+    (in_bom yes) (on_board yes)
+    (property "Reference" "G1" (id 0) (at 279.4 161.29 0)
+      (effects (font (size 1.27 1.27)) (justify left))
+    )
+    (property "Value" "LOGO" (id 1) (at 278.13 163.83 0)
+      (effects (font (size 1.27 1.27)) (justify left))
+    )
+    (property "Footprint" "eurovibes:LOGO" (id 2) (at 280.67 158.75 0)
+      (effects (font (size 1.27 1.27)) hide)
+    )
+    (property "Datasheet" "https://github.com/eurovibes" (id 3) (at 280.67 166.37 0)
+      (effects (font (size 1.27 1.27)) hide)
+    )
   )
   (symbol (lib_id "power:GND") (at 266.7 66.04 0) (unit 1)
@@
     )
     (pin "1")
+  )
+  (symbol (lib_id "Graphic:Logo_Open_Hardware_Small") (at 266.7 173.99 0) (unit 1)
+    (in_bom yes) (on_board yes) (fields_autoplaced)
+    (property "Reference" "#LOGO1" (id 0) (at 266.7 167.005 0)
+      (effects (font (size 1.27 1.27)) hide)
+    )
+    (property "Value" "Logo_Open_Hardware_Small" (id 1) (at 266.7 179.705 0)
+      (effects (font (size 1.27 1.27)) hide)
+    )
+    (property "Footprint" "" (id 2) (at 266.7 173.99 0)
+      (effects (font (size 1.27 1.27)) hide)
+    )
+    (property "Datasheet" "~" (id 3) (at 266.7 173.99 0)
+      (effects (font (size 1.27 1.27)) hide)
+    )
   )
   (symbol (lib_id "power:GND") (at 254 66.04 0) (unit 1)
@@
       (reference "#FLG0402") (unit 1) (value "PWR_FLAG") (footprint "")
     )
+    (path "/8a7ea79d-feb5-4c91-ad58-4466a260edea"
+      (reference "#LOGO1") (unit 1) (value "Logo_Open_Hardware_Small") (footprint "")
+    )
     (path "/b37654f6-617e-4451-b95f-b8693048d0c9"
       (reference "#PWR0101") (unit 1) (value "+3V3") (footprint "")
@@
       (reference "D316") (unit 1) (value "1N4148WT") (footprint "Diode_SMD:D_SOD-523")
     )
+    (path "/014897dd-0f3f-4c0f-8a32-f0744c0eb01e"
+      (reference "G1") (unit 1) (value "LOGO") (footprint "eurovibes:LOGO")
+    )
     (path "/6b131795-dcb5-484b-a4b3-38c0db9d2b44"
